File: boards/EltekFlatpack2-panel.kicad_pcb (KiCad board)
At the start: 2 copper layers, 92.5 x 96.2 mm, 179 parts, among them T1 Keystone 4912, T2 Keystone 4912

Commit message: Deploying to gh-pages from @ neg2led/flatpack2-adapter@9cc55d8c0d7576d7c777d3bbf8ae3edbd7cdf46f 🚀
Parts:
- removed the JP1 at (121.3, 83.0)
- removed the REF** at (60.0, 136.3) (x2)
- removed the REF** at (132.5, 45.0) (x2)
- removed the REF** at (60.0, 45.0) (x2)
- added REF**: NPTH, NPTH, F.Cu at (94.0, 106.0)
- added REF**: Fiducial, Fiducial, B.Cu at (60.0, 136.3)
- added REF**: Fiducial, Fiducial, F.Cu at (60.0, 136.3)
- added REF**: Fiducial, Fiducial, B.Cu at (132.5, 45.0)
- added REF**: Fiducial, Fiducial, F.Cu at (132.5, 45.0)
- added REF**: Fiducial, Fiducial, B.Cu at (60.0, 45.0)
- added REF**: Fiducial, Fiducial, F.Cu at (60.0, 45.0)
- JP1: renamed from REF**; value NPTH -> CTRL_VBUS+; footprint NPTH -> Jumper:SolderJumper-2_P1.3mm_Open_RoundedPad1.0x1.5mm
- moved JP1 35.7 mm to (121.3, 83.0), turned to 270 degrees
