File: boards/EltekFlatpack2.kicad_pcb (KiCad board)
At the start: 2 copper layers, 43.8 x 81 mm, 17 parts, among them T1 Keystone 4912, T2 Keystone 4912

Commit message: Deploying to gh-pages from @ neg2led/flatpack2-adapter@9cc55d8c0d7576d7c777d3bbf8ae3edbd7cdf46f 🚀
Parts:
- removed the T2 at (153.6, 70.2)
- added H4: M3, MountingHole:MountingHole_2.7mm_M2.5_ISO7380_Pad_TopBottom, F.Cu at (169.1, 62.2)
- T2: renamed from H4; value M3 -> Keystone 4912; footprint MountingHole:MountingHole_2.7mm_M2.5_ISO7380_Pad_TopBottom -> 1 My Footprints:Connector_Keystone_4912_Overlaid
- moved T2 17.5 mm to (153.6, 70.2), turned to 90 degrees
Connections:
- T2 pad 1: Board_1-Earth -> Board_1-/VBUS-
